Commit message: 021223

File: src/kssbot/kssbot_description/ros2_control/kssbot.ros2_control.xacro (robot description, xacro)
@@ -2,4 +2,29 @@
 <robot xmlns:xacro="http://www.ros.org/wiki/xacro">
   <xacro:macro name="kssbot_ros2_control" params="name prefix">
+        <ros2_control name="${name}" type="system">
+            <hardware>
+                <plugin>kssbot_hardware/kssbot_diffdrive_rasp4</plugin>
+                <param name="left_wheel_name">left_wheel_joint</param>
+                <param name="right_wheel_name">right_wheel_joint</param>
+                <param name="loop_rate">30</param>
+            </hardware>
+            <joint name="left_wheel_joint">
+                <command_interface name="velocity">
+                    <param name="min">-10</param>
+                    <param name="max">10</param>
+                </command_interface>
+                <state_interface name="position"/>
+                <state_interface name="velocity"/>
+            </joint>
+            <joint name="right_wheel_joint">
+                <command_interface name="velocity">
+                    <param name="min">-10</param>
+                    <param name="max">10</param>
+                </command_interface>
+                <state_interface name="position"/>
+                <state_interface name="velocity"/>
+            </joint>
+        </ros2_control>
+<!--
     <ros2_control name="${name}" type="system">
       <hardware>
@@ -8,5 +33,5 @@
         <param name="example_param_hw_stop_duration_sec">3.0</param>
       </hardware>
-      <joint name="${prefix}left_wheel_joint">
+      <joint name="left_wheel_joint">
         <command_interface name="velocity"/>
           <param name = 'min'>-10</param>
@@ -15,5 +40,5 @@
         <state_interface name="velocity"/>
       </joint>
-      <joint name="${prefix}right_wheel_joint">
+      <joint name="right_wheel_joint">
         <command_interface name="velocity"/>
           <param name = 'min'>-10</param>
@@ -23,4 +48,5 @@
       </joint>
     </ros2_control>
+-->
   </xacro:macro>
 </robot>

Commit message: 0426

File: src/kssbot/kssbot_description/ros2_control/kssbot.ros2_control.xacro (robot description, xacro)
@@ -2,5 +2,5 @@
 <robot xmlns:xacro="http://www.ros.org/wiki/xacro">
   <xacro:macro name="kssbot_ros2_control" params="name prefix">
-        <ros2_control name="${name}" type="system">
+        <ros2_control name="kssbot_diffdrive" type="system">
             <hardware>
                 <plugin>kssbot_hardware/kssbot_diffdrive_rasp4</plugin>

File: src/kssbot/kssbot_description/urdf/kssbot_description.urdf.xacro (robot description, xacro)
@@ -4,16 +4,28 @@
   <!-- Constants for robot dimensions -->
   <xacro:property name="PI" value="3.1415926535897931"/>
-  <xacro:property name="base_mass" value="0.1" /> <!-- arbitrary value for base mass -->
+  <!-- arbitrary value for base mass -->
+  <xacro:property name="base_mass" value="0.1" />
   <xacro:property name="base_width" value="0.12" />
   <xacro:property name="base_length" value="0.12" />
-  <xacro:property name="base_height" value="0.07" />
-  <xacro:property name="wheel_mass" value="0.05" /> <!-- arbitrary value for wheel mass -->
-  <xacro:property name="wheel_len" value="0.025" />
+  <xacro:property name="base_height" value="0.065" />
+  <xacro:property name="base_offset" value="0.02" />
+  <!-- arbitrary value for wheel mass -->
+  <xacro:property name="wheel_mass" value="0.05" />
+  <xacro:property name="wheel_len" value="0.024" />
   <xacro:property name="wheel_radius" value="0.035" />
-  <xacro:property name="caster_wheel_mass" value="0.1" /> <!-- arbitrary value for caster wheel mass -->
+  <!-- arbitrary value for caster wheel mass -->
+  <xacro:property name="caster_wheel_mass" value="0.1" />
   <xacro:property name="caster_wheel_radius" value="0.015" />
-  <xacro:property name="z_offset" value="0.02" /> <!-- Space btw top of beam and the each joint -->
+  <!-- Space btw top of beam and the each joint -->
+  <xacro:property name="z_offset" value="${base_height/2}" />
   <!-- Base Link -->
   <link name="${prefix}base_link">
+    <visual>
+      <origin xyz="0 0 ${base_offset + z_offset}" rpy="0 0 0"/>
+      <geometry>
+        <box size="${base_width} ${base_length} ${base_height}"/>
+      </geometry>
+      <material name="orange"/>
+    </visual>
     <collision>
       <origin xyz="0 0 0" rpy="0 0 0"/>
@@ -22,118 +34,85 @@
       </geometry>
     </collision>
+    <inertial>
+      <origin xyz="0 0 0" rpy="0 0 0"/>
+      <mass value="${base_mass}"/>
+      <inertia
+        ixx="${base_mass / 12.0 * (base_length*base_length + base_height*base_height)}" ixy="0.0" ixz="0.0"
+        iyy="${base_mass / 12.0 * (base_height*base_height + base_width*base_width)}" iyz="0.0"
+        izz="${base_mass / 12.0 * (base_width*base_width + base_length*base_length)}"/>
+    </inertial>
+  </link>
+  <!-- left wheel Joint -->
+    <joint name="${prefix}left_wheel_joint" type="continuous">
+    <parent link="${prefix}base_link"/>
+    <child link="${prefix}left_wheel"/>
+    <origin xyz="0.025 -${base_width/2 + wheel_len/2} ${wheel_radius}" rpy="0 0 0"/>
+    <axis xyz="0 1 0"/>
+    <dynamics damping="0.2"/>
+  </joint>
+  <!-- left wheel Link -->
+  <link name="${prefix}left_wheel">
+    <collision>
+      <origin xyz="0 0 0" rpy="0 0 0"/>
+      <geometry>
+        <cylinder length="${wheel_len}" radius="${wheel_radius}"/>
+      </geometry>
+    </collision>
     <visual>
-      <origin xyz="0 0 ${z_offset}" rpy="0 0 0"/>
+      <origin xyz="0 0 0" rpy="${pi/2} 0 0"/>
       <geometry>
-        <box size="${base_width} ${base_length} ${base_height}"/>
+        <cylinder length="${wheel_len}" radius="${wheel_radius}"/>
       </geometry>
-      <material name="orange"/>
+      <material name="black"/>
     </visual>
     <inertial>
       <origin xyz="0 0 0" rpy="0 0 0"/>
-      <mass value="${base_mass}"/>
-      <inertiaz_offset
-        ixx="${base_mass / 12.0 * (base_length*base_length + base_height*base_height)}" ixy="0.0" ixz="0.0"
-        iyy="${base_mass / 12.0 * (base_height*base_height + base_width*base_width)}" iyz="0.0"
-        izz="${base_mass / 12.0 * (base_width*base_width + base_length*base_length)}"/>
+      <mass value="${wheel_mass}"/>
+      <inertia
+        ixx="${wheel_mass / 12.0 * (3*wheel_radius + wheel_len*wheel_len)}" ixy="0.0" ixz="0.0"
+        iyy="${wheel_mass / 12.0 * wheel_radius*wheel_radius}" iyz="0.0"
+        izz="${wheel_mass / 12.0 * wheel_radius*wheel_radius}"/>
       </inertial>
-    </link>
-    <joint name="${prefix}left_wheel_joint" type="continuous">
-      <parent link="${prefix}base_link"/>
-      <child link="${prefix}left_wheel"/>
-      <origin xyz="0.025 -${base_width/2} ${z_offset}" rpy="0 0 0"/>
-      <axis xyz="0 1 0"/>
-      <dynamics damping="0.2"/>
-    </joint>
-    <!-- left wheel Link -->
-    <link name="${prefix}left_wheel">
-      <collision>
-        <origin xyz="0 0 0" rpy="${PI/2} 0 0"/>
-        <geometry>
-          <cylinder length="${wheel_len}" radius="${wheel_radius}"/>
-        </geometry>
-      </collision>
-      <visual>
-        <origin xyz="0 0 0" rpy="${PI/2} 0 0"/>
-        <geometry>
-          <cylinder length="${wheel_len}" radius="${wheel_radius}"/>
-        </geometry>
-        <material name="black"/>
-      </visual>
-      <inertial>
-        <origin xyz="0 0 0" rpy="${PI/2} 0 0"/>
-        <mass value="${wheel_mass}"/>
-        <inertia
-          ixx="${wheel_mass / 12.0 * (3*wheel_radius + wheel_len*wheel_len)}" ixy="0.0" ixz="0.0"
-          iyy="${wheel_mass / 12.0 * wheel_radius*wheel_radius}" iyz="0.0"
-          izz="${wheel_mass / 12.0 * wheel_radius*wheel_radius}"/>
-        </inertial>
-      </link>
+  </link>
+  <!-- right wheel Joint -->
     <joint name="${prefix}right_wheel_joint" type="continuous">
-      <parent link="${prefix}base_link"/>
-      <child link="${prefix}right_wheel"/>
-      <origin xyz="0 ${base_width/2} ${z_offset}" rpy="0 0 0"/>
-      <axis xyz="0 1 0"/>
-      <dynamics damping="0.2"/>
-    </joint>
-    <!-- right wheel Link -->
-    <link name="${prefix}right_wheel">
-      <collision>
-        <origin xyz="0 0 0" rpy="${PI/2} 0 0"/>
-        <geometry>
-          <cylinder length="${wheel_len}" radius="${wheel_radius}"/>
-        </geometry>
-      </collision>
-      <visual>
-        <origin xyz="0 0 0" rpy="${PI/2} 0 0"/>
-        <geometry>
-          <cylinder length="${wheel_len}" radius="${wheel_radius}"/>
-        </geometry>
-        <material name="black"/>
-      </visual>
-      <inertial>
-        <origin xyz="0 0 0" rpy="${PI/2} 0 0"/>
-        <mass value="${wheel_mass}"/>
-        <inertia
-          ixx="${wheel_mass / 12.0 * (3*wheel_radius + wheel_len*wheel_len)}" ixy="0.0" ixz="0.0"
-          iyy="${wheel_mass / 12.0 * wheel_radius*wheel_radius}" iyz="0.0"
-          izz="${wheel_mass / 12.0 * wheel_radius*wheel_radius}"/>
-        </inertial>
-      </link>
-    <joint name="${prefix}caster_frontal_wheel_joint" type="fixed">
+    <parent link="${prefix}base_link"/>
+    <child link="${prefix}right_wheel"/>
+    <origin xyz="0.025 ${base_width/2 + wheel_len/2} ${wheel_radius}" rpy="0 0 0"/>
+    <axis xyz="0 1 0"/>
+    <dynamics damping="0.2"/>
+  </joint>
+  <!-- right wheel Link -->
+  <link name="${prefix}right_wheel">
+    <collision>
+      <origin xyz="0 0 0" rpy="0 0 0"/>
+      <geometry>
+        <cylinder length="${wheel_len}" radius="${wheel_radius}"/>
+      </geometry>
+    </collision>
+    <visual>
+      <origin xyz="0 0 0" rpy="${pi/2} 0 0"/>
+      <geometry>
+        <cylinder length="${wheel_len}" radius="${wheel_radius}"/>
+      </geometry>
+      <material name="black"/>
+    </visual>
+    <inertial>
+      <origin xyz="0 0 0" rpy="0 0 0"/>
+      <mass value="${wheel_mass}"/>
+      <inertia
+        ixx="${wheel_mass / 12.0 * (3*wheel_radius + wheel_len*wheel_len)}" ixy="0.0" ixz="0.0"
+        iyy="${wheel_mass / 12.0 * wheel_radius*wheel_radius}" iyz="0.0"
+        izz="${wheel_mass / 12.0 * wheel_radius*wheel_radius}"/>
+      </inertial>
+  </link>
+    <!-- footprint caster Joint -->
+    <joint name="${prefix}footprint_joint" type="fixed">
       <parent link="${prefix}base_link"/>
       <child link="${prefix}caster_frontal_wheel"/>
       <origin xyz="${base_width/2 - caster_wheel_radius} 0 ${z_offset}" rpy="0 0 0"/>
     </joint>
-    <!-- caster frontal wheel Link -->
+    <!-- footprint caster Link -->
     <link name="${prefix}caster_frontal_wheel">
-      <collision>
-        <origin xyz="0 0 0" rpy="0 0 0"/>
-        <geometry>
-          <sphere radius="${caster_wheel_radius}"/>
-        </geometry>
-      </collision>
-      <visual>
-        <origin xyz="0 0 0" rpy="0 0 0"/>
-        <geometry>
-          <sphere radius="${caster_wheel_radius}"/>
-        </geometry>
-        <material name="white"/>
-      </visual>
-      <inertial>
-        <origin xyz="0 0 0" rpy="0 0 0"/>
-        <mass value="${caster_wheel_mass}"/>
-        <inertia
-          ixx="${caster_wheel_mass * 0.4 * (caster_wheel_radius * caster_wheel_radius)}" ixy="0.0" ixz="0.0"
-          iyy="${caster_wheel_mass * 0.4 * (caster_wheel_radius * caster_wheel_radius)}" iyz="0.0"
-          izz="${caster_wheel_mass * 0.4 * (caster_wheel_radius * caster_wheel_radius)}"/>
-        </inertial>
-      </link>
-    <joint name="${prefix}caster_rear_wheel_joint" type="fixed">
-      <parent link="${prefix}base_link"/>
-      <child link="${prefix}caster_rear_wheel"/>
-      <origin xyz="${-base_width/2 + caster_wheel_radius} 0 ${z_offset}" rpy="0 0 0"/>
-    </joint>
-    <!-- caster rear wheel Link -->
-    <link name="${prefix}caster_rear_wheel">
       <collision>
         <origin xyz="0 0 0" rpy="0 0 0"/>

Commit message: 042923

File: src/kssbot/kssbot_description/ros2_control/kssbot.ros2_control.xacro (robot description, xacro)
@@ -8,4 +8,5 @@
                 <param name="right_wheel_name">right_wheel_joint</param>
                 <param name="loop_rate">30</param>
+                <!-- add params here -->
             </hardware>
             <joint name="left_wheel_joint">

File: src/kssbot/kssbot_description/urdf/kssbot_description.urdf.xacro (robot description, xacro)
@@ -4,32 +4,59 @@
   <!-- Constants for robot dimensions -->
   <xacro:property name="PI" value="3.1415926535897931"/>
-  <!-- arbitrary value for base mass -->
-  <xacro:property name="base_mass" value="0.1" />
+  <!-- arbitrary value for base value -->
+  <xacro:property name="base_mass" value="0.06" />
+  <xacro:property name="base_length" value="0.12" />
   <xacro:property name="base_width" value="0.12" />
-  <xacro:property name="base_length" value="0.12" />
   <xacro:property name="base_height" value="0.065" />
   <xacro:property name="base_offset" value="0.02" />
-  <!-- arbitrary value for wheel mass -->
-  <xacro:property name="wheel_mass" value="0.05" />
+  <!-- arbitrary value for wheel value -->
+  <xacro:property name="wheel_mass" value="0.06" />
   <xacro:property name="wheel_len" value="0.024" />
   <xacro:property name="wheel_radius" value="0.035" />
-  <!-- arbitrary value for caster wheel mass -->
+  <!-- arbitrary value for caster wheel value -->
   <xacro:property name="caster_wheel_mass" value="0.1" />
   <xacro:property name="caster_wheel_radius" value="0.015" />
   <!-- Space btw top of beam and the each joint -->
   <xacro:property name="z_offset" value="${base_height/2}" />
+  <!-- arbitrary value for ultrasonic eye value -->
+  <xacro:property name="sonic_mass" value="0.06" />
+  <xacro:property name="sonic_len" value="0.007" />
+  <xacro:property name="sonic_radius" value="0.0075" />
+  <!-- arbitrary value for front camera value -->
+  <xacro:property name="cam_length" value="0.02" />
+  <xacro:property name="cam_width" value="0.045" />
+  <xacro:property name="cam_height" value="0.033" />
   <!-- Base Link -->
-  <link name="${prefix}base_link">
-    <visual>
-      <origin xyz="0 0 ${base_offset + z_offset}" rpy="0 0 0"/>
-      <geometry>
-        <box size="${base_width} ${base_length} ${base_height}"/>
-      </geometry>
-      <material name="orange"/>
-    </visual>
-    <collision>
-      <origin xyz="0 0 0" rpy="0 0 0"/>
-      <geometry>
-        <box size="${base_width} ${base_length} ${base_height}"/>
+  <link
+    name="${prefix}base_link">
+  </link>
+  <!-- Base Footprint Joint -->
+  <joint name="base_footprint_joint" type="fixed">
+      <parent link="${prefix}base_link"/>
+      <child link="${prefix}base_footprint"/>
+      <origin xyz="0 0 0" rpy="0 0 0"/>
+  </joint>
+  <link
+    name="${prefix}base_footprint">
+  </link>
+  <!-- Chassis Joint -->
+  <joint name="${prefix}chassis_joint" type="fixed">
+      <parent link="${prefix}base_link"/>
+      <child link="${prefix}chassis"/>
+      <origin xyz="0 0 ${base_offset + z_offset}"/>
+  </joint>
+  <!-- Chassis Link-->
+  <link name="${prefix}chassis">
+    <visual>
+      <origin xyz="0 0 0" rpy="0 0 0"/>
+      <geometry>
+        <box size="${base_length} ${base_width} ${base_height}"/>
+      </geometry>
+      <material name="black"/>
+    </visual>
+    <collision>
+      <origin xyz="0 0 0" rpy="0 0 0"/>
+      <geometry>
+        <box size="${base_length} ${base_width} ${base_height}"/>
       </geometry>
     </collision>
@@ -45,7 +72,7 @@
   <!-- left wheel Joint -->
     <joint name="${prefix}left_wheel_joint" type="continuous">
-    <parent link="${prefix}base_link"/>
+    <parent link="${prefix}chassis"/>
     <child link="${prefix}left_wheel"/>
-    <origin xyz="0.025 -${base_width/2 + wheel_len/2} ${wheel_radius}" rpy="0 0 0"/>
+    <origin xyz="0.035 ${base_width/2 + wheel_len/2} ${base_offset-wheel_radius}" rpy="0 0 0"/>
     <axis xyz="0 1 0"/>
     <dynamics damping="0.2"/>
@@ -64,5 +91,37 @@
         <cylinder length="${wheel_len}" radius="${wheel_radius}"/>
       </geometry>
-      <material name="black"/>
+      <material name="orange"/>
+    </visual>
+    <inertial>
+      <origin xyz="0 0 0" rpy="0 0 0"/>
+      <mass value="${wheel_mass}"/>
+      <inertia
+        ixx="${wheel_mass / 12.0 * (3*wheel_radius + wheel_len*wheel_len)}" ixy="0.0" ixz="0.0"
+        iyy="${wheel_mass / 12.0 * wheel_radius*wheel_radius}" iyz="0.0"
+        izz="${wheel_mass / 12.0 * wheel_radius*wheel_radius}"/>
+      </inertial>
+  </link>
+  <!-- left wheel dummy Joint -->
+  <joint name="${prefix}left_wheel_dummy_joint" type="fixed">
+    <parent link="${prefix}chassis"/>
+    <child link="${prefix}left_wheel_dummy"/>
+    <origin xyz="-0.055 ${base_width/2 + wheel_len/2} ${base_offset-wheel_radius}" rpy="0 0 0"/>
+    <axis xyz="0 1 0"/>
+    <dynamics damping="0.2"/>
+  </joint>
+  <!-- left wheel dummy Link -->
+  <link name="${prefix}left_wheel_dummy">
+    <collision>
+      <origin xyz="0 0 0" rpy="0 0 0"/>
+      <geometry>
+        <cylinder length="${wheel_len}" radius="${wheel_radius}"/>
+      </geometry>
+    </collision>
+    <visual>
+      <origin xyz="0 0 0" rpy="${pi/2} 0 0"/>
+      <geometry>
+        <cylinder length="${wheel_len}" radius="${wheel_radius}"/>
+      </geometry>
+      <material name="orange"/>
     </visual>
     <inertial>
@@ -77,7 +136,7 @@
   <!-- right wheel Joint -->
     <joint name="${prefix}right_wheel_joint" type="continuous">
-    <parent link="${prefix}base_link"/>
+    <parent link="${prefix}chassis"/>
     <child link="${prefix}right_wheel"/>
-    <origin xyz="0.025 ${base_width/2 + wheel_len/2} ${wheel_radius}" rpy="0 0 0"/>
+    <origin xyz="0.035 -${base_width/2 + wheel_len/2} ${base_offset-wheel_radius}" rpy="0 0 0"/>
     <axis xyz="0 1 0"/>
     <dynamics damping="0.2"/>
@@ -96,27 +155,107 @@
         <cylinder length="${wheel_len}" radius="${wheel_radius}"/>
       </geometry>
-      <material name="black"/>
-    </visual>
-    <inertial>
-      <origin xyz="0 0 0" rpy="0 0 0"/>
-      <mass value="${wheel_mass}"/>
-      <inertia
-        ixx="${wheel_mass / 12.0 * (3*wheel_radius + wheel_len*wheel_len)}" ixy="0.0" ixz="0.0"
-        iyy="${wheel_mass / 12.0 * wheel_radius*wheel_radius}" iyz="0.0"
-        izz="${wheel_mass / 12.0 * wheel_radius*wheel_radius}"/>
-      </inertial>
-  </link>
-    <!-- footprint caster Joint -->
-    <joint name="${prefix}footprint_joint" type="fixed">
-      <parent link="${prefix}base_link"/>
-      <child link="${prefix}caster_frontal_wheel"/>
-      <origin xyz="${base_width/2 - caster_wheel_radius} 0 ${z_offset}" rpy="0 0 0"/>
+      <material name="orange"/>
+    </visual>
+    <inertial>
+      <origin xyz="0 0 0" rpy="0 0 0"/>
+      <mass value="${wheel_mass}"/>
+      <inertia
+        ixx="${wheel_mass / 12.0 * (3*wheel_radius + wheel_len*wheel_len)}" ixy="0.0" ixz="0.0"
+        iyy="${wheel_mass / 12.0 * wheel_radius*wheel_radius}" iyz="0.0"
+        izz="${wheel_mass / 12.0 * wheel_radius*wheel_radius}"/>
+      </inertial>
+  </link>
+<!-- right wheel dummy Joint -->
+    <joint name="${prefix}right_wheel_dummy_joint" type="fixed">
+    <parent link="${prefix}chassis"/>
+    <child link="${prefix}right_wheel_dummy"/>
+    <origin xyz="-0.055 -${base_width/2 + wheel_len/2} ${base_offset-wheel_radius}" rpy="0 0 0"/>
+    <axis xyz="0 1 0"/>
+    <dynamics damping="0.2"/>
+  </joint>
+  <!-- right wheel dummy Link -->
+  <link name="${prefix}right_wheel_dummy">
+    <collision>
+      <origin xyz="0 0 0" rpy="0 0 0"/>
+      <geometry>
+        <cylinder length="${wheel_len}" radius="${wheel_radius}"/>
+      </geometry>
+    </collision>
+    <visual>
+      <origin xyz="0 0 0" rpy="${pi/2} 0 0"/>
+      <geometry>
+        <cylinder length="${wheel_len}" radius="${wheel_radius}"/>
+      </geometry>
+      <material name="orange"/>
+    </visual>
+    <inertial>
+      <origin xyz="0 0 0" rpy="0 0 0"/>
+      <mass value="${wheel_mass}"/>
+      <inertia
+        ixx="${wheel_mass / 12.0 * (3*wheel_radius + wheel_len*wheel_len)}" ixy="0.0" ixz="0.0"
+        iyy="${wheel_mass / 12.0 * wheel_radius*wheel_radius}" iyz="0.0"
+        izz="${wheel_mass / 12.0 * wheel_radius*wheel_radius}"/>
+      </inertial>
+  </link>
+  <!-- left ultrasonic eye Joint -->
+    <joint name="${prefix}left_ultrasonic_eye_joint" type="fixed">
+    <parent link="${prefix}chassis"/>
+    <child link="${prefix}left_ultrasonic_eye"/>
+    <origin xyz="0.06 0.0125 -0.0125" rpy="0 0 0"/>
+    <axis xyz="0 1 0"/>
+    <dynamics damping="0.2"/>
+  </joint>
+  <!-- left ultrasonic eye Link -->
+  <link name="${prefix}left_ultrasonic_eye">
+    <collision>
+      <origin xyz="0 0 0" rpy="0 0 0"/>
+      <geometry>
+        <cylinder length="0.007" radius="0.0075"/>
+      </geometry>
+    </collision>
+    <visual>
+      <origin xyz="0 0 0" rpy="0 ${pi/2} 0"/>
+      <geometry>
+        <cylinder length="${sonic_len}" radius="${sonic_radius}"/>
+      </geometry>
+      <material name="grey"/>
+    </visual>
+  </link>
+  <!-- right ultrasonic eye Joint -->
+  <joint name="${prefix}right_ultrasonic_eye_joint" type="fixed">
+    <parent link="${prefix}chassis"/>
+    <child link="${prefix}right_ultrasonic_eye"/>
+    <origin xyz="0.06 -0.0125 -0.0125" rpy="0 0 0"/>
+    <axis xyz="0 1 0"/>
+    <dynamics damping="0.2"/>
+  </joint>
+  <!-- right ultrasonic eye Link -->
+  <link name="${prefix}right_ultrasonic_eye">
+    <collision>
+      <origin xyz="0 0 0" rpy="0 0 0"/>
+      <geometry>
+        <cylinder length="${sonic_len}" radius="${sonic_radius}"/>
+      </geometry>
+    </collision>
+    <visual>
+      <origin xyz="0 0 0" rpy="0 ${pi/2} 0"/>
+      <geometry>
+        <cylinder length="0.007" radius="0.0075"/>
+      </geometry>
+      <material name="grey"/>
+    </visual>
+  </link>
+    <!-- front camera Joint -->
+    <joint name="${prefix}front_camera_joint" type="fixed">
+      <parent link="${prefix}chassis"/>
+      <child link="${prefix}front_camera"/>
+      <origin xyz="0.06 0 0.0225" rpy="0 0 0"/>
     </joint>
-    <!-- footprint caster Link -->
-    <link name="${prefix}caster_frontal_wheel">
+    <!-- front camera Link -->
+    <link name="${prefix}front_camera">
       <collision>
         <origin xyz="0 0 0" rpy="0 0 0"/>
         <geometry>
-          <sphere radius="${caster_wheel_radius}"/>
+          <box size="${cam_length} ${cam_width} ${cam_height}"/>
         </geometry>
       </collision>
@@ -124,17 +263,9 @@
         <origin xyz="0 0 0" rpy="0 0 0"/>
         <geometry>
-          <sphere radius="${caster_wheel_radius}"/>
+         <box size="${cam_length} ${cam_width} ${cam_height}"/>
         </geometry>
-        <material name="white"/>
+        <material name="red"/>
       </visual>
-      <inertial>
-        <origin xyz="0 0 0" rpy="0 0 0"/>
-        <mass value="${caster_wheel_mass}"/>
-        <inertia
-          ixx="${caster_wheel_mass * 0.4 * (caster_wheel_radius * caster_wheel_radius)}" ixy="0.0" ixz="0.0"
-          iyy="${caster_wheel_mass * 0.4 * (caster_wheel_radius * caster_wheel_radius)}" iyz="0.0"
-          izz="${caster_wheel_mass * 0.4 * (caster_wheel_radius * caster_wheel_radius)}"/>
-        </inertial>
-      </link>
+    </link>
   </xacro:macro>
 </robot>
