Commit message: 050823

File: src/kssbot/kssbot_description/ros2_control/kssbot.ros2_control.xacro (robot description, xacro)
@@ -2,11 +2,35 @@
 <robot xmlns:xacro="http://www.ros.org/wiki/xacro">
   <xacro:macro name="kssbot_ros2_control" params="name prefix">
+      <xacro:unless value="$(arg sim_mode)">
         <ros2_control name="kssbot_diffdrive" type="system">
+          <hardware>
+            <plugin>kssbot_hardware/kssbot_diffdrive_rasp4</plugin>
+            <param name="left_wheel_name">left_wheel_joint</param>
+            <param name="right_wheel_name">right_wheel_joint</param>
+            <param name="loop_rate">30</param>
+            <!-- add params here -->
+          </hardware>
+          <joint name="left_wheel_joint">
+            <command_interface name="velocity">
+              <param name="min">-10</param>
+              <param name="max">10</param>
+            </command_interface>
+            <state_interface name="position"/>
+            <state_interface name="velocity"/>
+          </joint>
+          <joint name="right_wheel_joint">
+            <command_interface name="velocity">
+              <param name="min">-10</param>
+              <param name="max">10</param>
+            </command_interface>
+            <state_interface name="position"/>
+            <state_interface name="velocity"/>
+          </joint>
+        </ros2_control>
+      </xacro:unless>
+      <xacro:if value="$(arg sim_mode)">
+        <ros2_control name="GazeboSystem" type="system">
             <hardware>
-                <plugin>kssbot_hardware/kssbot_diffdrive_rasp4</plugin>
-                <param name="left_wheel_name">left_wheel_joint</param>
-                <param name="right_wheel_name">right_wheel_joint</param>
-                <param name="loop_rate">30</param>
-                <!-- add params here -->
+                <plugin>gazebo_ros2_control/GazeboSystem</plugin>
             </hardware>
             <joint name="left_wheel_joint">
@@ -15,6 +39,6 @@
                     <param name="max">10</param>
                 </command_interface>
+                <state_interface name="velocity"/>
                 <state_interface name="position"/>
-                <state_interface name="velocity"/>
             </joint>
             <joint name="right_wheel_joint">
@@ -23,9 +47,15 @@
                     <param name="max">10</param>
                 </command_interface>
+                <state_interface name="velocity"/>
                 <state_interface name="position"/>
-                <state_interface name="velocity"/>
             </joint>
         </ros2_control>
-<!--
+      </xacro:if>
+      <gazebo>
+        <plugin name="gazebo_ros2_control" filename="libgazebo_ros2_control.so">
+          <parameters>$(find kssbot_bringup)/config/kssbot_sim.controllers.yaml</parameters>
+        </plugin>
+      </gazebo>
+    <!--
     <ros2_control name="${name}" type="system">
       <hardware>
@@ -48,6 +78,5 @@
         <state_interface name="velocity"/>
       </joint>
-    </ros2_control>
--->
+    </ros2_control> -->
   </xacro:macro>
 </robot>

File: src/kssbot/kssbot_description/urdf/kssbot.urdf.xacro (robot description, xacro)
@@ -1,12 +1,26 @@
 <?xml version="1.0"?>
-<!-- Basic differential drive mobile base -->
-<robot xmlns:xacro="http://www.ros.org/wiki/xacro" name="diffdrive_robot">
+<robot xmlns:xacro="http://www.ros.org/wiki/xacro" name="kssbot">
   <xacro:arg name="prefix" default="" />
+  <xacro:arg name="use_ros2_control" default="true"/>
+  <xacro:arg name="sim_mode" default="false"/>
+  <!-- Basic differential drive mobile base -->
   <xacro:include filename="$(find kssbot_description)/urdf/kssbot_description.urdf.xacro" />
   <!-- Import Rviz colors -->
-  <xacro:include filename="$(find kssbot_description)/gazebo/kssbot.materials.xacro" />
+  <xacro:include filename="$(find kssbot_description)/urdf/kssbot.materials.xacro" />
   <!-- Import kssbot ros2_control description -->
-  <xacro:include filename="$(find kssbot_description)/ros2_control/kssbot.ros2_control.xacro" />
-  <xacro:kssbot prefix="$(arg prefix)" />
-  <xacro:kssbot_ros2_control name="kssBot" prefix="$(arg prefix)" />
+  <!-- if use ros2_control  -->
+  <xacro:if value="$(arg use_ros2_control)">
+    <xacro:include filename="$(find kssbot_description)/ros2_control/kssbot.ros2_control.xacro" />
+    <!-- this line is for urdf reading(kssbot_description.urdf.xacro) -->
+    <xacro:kssbot prefix="$(arg prefix)" />
+    <!-- this line is for ros2_control reading(kssbot.ros2_control.xacro) -->
+    <xacro:kssbot_ros2_control name="kssBot" prefix="$(arg prefix)" />
+  </xacro:if>
+  <!-- if use gazebo  -->
+  <xacro:unless value="$(arg use_ros2_control)">
+    <xacro:include filename="$(find kssbot_description)/ros2_control/kssbot.gazebo.xacro" />
+  </xacro:unless>
+  <!-- Add addtional component description -->
+  <!-- <xacro:include filename="lidar.xacro" /> -->
+  <!-- <xacro:include filename="camera.xacro" /> -->
 </robot>

File: src/kssbot/kssbot_description/urdf/kssbot_description.urdf.xacro (robot description, xacro)
@@ -2,253 +2,253 @@
 <robot xmlns:xacro="http://www.ros.org/wiki/xacro">
   <xacro:macro name="kssbot" params="prefix">
-  <!-- Constants for robot dimensions -->
-  <xacro:property name="PI" value="3.1415926535897931"/>
-  <!-- arbitrary value for base value -->
-  <xacro:property name="base_mass" value="0.1" />
-  <xacro:property name="base_length" value="0.12" />
-  <xacro:property name="base_width" value="0.12" />
-  <xacro:property name="base_height" value="0.065" />
-  <xacro:property name="base_offset" value="0.02" />
-  <!-- arbitrary value for wheel value -->
-  <xacro:property name="wheel_mass" value="0.06" />
-  <xacro:property name="wheel_len" value="0.024" />
-  <xacro:property name="wheel_radius" value="0.035" />
-  <!-- Space btw top of beam and the each joint -->
-  <xacro:property name="z_offset" value="${base_height/2}" />
-  <!-- arbitrary value for ultrasonic eye value -->
-  <xacro:property name="sonic_mass" value="0.06" />
-  <xacro:property name="sonic_len" value="0.007" />
-  <xacro:property name="sonic_radius" value="0.0075" />
-  <!-- arbitrary value for front camera value -->
-  <xacro:property name="cam_length" value="0.02" />
-  <xacro:property name="cam_width" value="0.045" />
-  <xacro:property name="cam_height" value="0.033" />
-  <!-- Base Link -->
-  <link
-    name="${prefix}base_link">
-  </link>
-  <!-- Base Footprint Joint -->
-  <joint name="base_footprint_joint" type="fixed">
-      <parent link="${prefix}base_link"/>
-      <child link="${prefix}base_footprint"/>
-      <origin xyz="0 0 0" rpy="0 0 0"/>
-  </joint>
-  <link
-    name="${prefix}base_footprint">
-  </link>
-  <!-- Chassis Joint -->
-  <joint name="${prefix}chassis_joint" type="fixed">
-      <parent link="${prefix}base_link"/>
-      <child link="${prefix}chassis"/>
-      <origin xyz="0 0 ${base_offset + z_offset}"/>
-  </joint>
-  <!-- Chassis Link-->
-  <link name="${prefix}chassis">
-    <visual>
-      <origin xyz="0 0 0" rpy="0 0 0"/>
-      <geometry>
-        <box size="${base_length} ${base_width} ${base_height}"/>
-      </geometry>
-      <material name="black"/>
-    </visual>
-    <collision>
-      <origin xyz="0 0 0" rpy="0 0 0"/>
-      <geometry>
-        <box size="${base_length} ${base_width} ${base_height}"/>
-      </geometry>
-    </collision>
-    <inertial>
-      <origin xyz="0 0 0" rpy="0 0 0"/>
-      <mass value="${base_mass}"/>
-      <inertia
-        ixx="${base_mass / 12.0 * (base_length*base_length + base_height*base_height)}" ixy="0.0" ixz="0.0"
-        iyy="${base_mass / 12.0 * (base_height*base_height + base_width*base_width)}" iyz="0.0"
-        izz="${base_mass / 12.0 * (base_width*base_width + base_length*base_length)}"/>
-    </inertial>
-  </link>
-  <!-- left wheel Joint -->
-    <joint name="${prefix}left_wheel_joint" type="continuous">
-    <parent link="${prefix}chassis"/>
-    <child link="${prefix}left_wheel"/>
-    <origin xyz="0.035 ${base_width/2 + wheel_len/2} ${base_offset-wheel_radius}" rpy="0 0 0"/>
-    <axis xyz="0 1 0"/>
-    <dynamics damping="0.2"/>
-  </joint>
-  <!-- left wheel Link -->
-  <link name="${prefix}left_wheel">
-    <collision>
-      <origin xyz="0 0 0" rpy="0 0 0"/>
-      <geometry>
-        <cylinder length="${wheel_len}" radius="${wheel_radius}"/>
-      </geometry>
-    </collision>
-    <visual>
-      <origin xyz="0 0 0" rpy="${pi/2} 0 0"/>
-      <geometry>
-        <cylinder length="${wheel_len}" radius="${wheel_radius}"/>
-      </geometry>
-      <material name="orange"/>
-    </visual>
-    <inertial>
-      <origin xyz="0 0 0" rpy="0 0 0"/>
-      <mass value="${wheel_mass}"/>
-      <inertia
-        ixx="${wheel_mass / 12.0 * (3*wheel_radius + wheel_len*wheel_len)}" ixy="0.0" ixz="0.0"
-        iyy="${wheel_mass / 12.0 * wheel_radius*wheel_radius}" iyz="0.0"
-        izz="${wheel_mass / 12.0 * wheel_radius*wheel_radius}"/>
+    <!-- Constants for robot dimensions -->
+    <xacro:property name="PI" value="3.1415926535897931"/>
+    <!-- arbitrary value for base value -->
+    <xacro:property name="base_mass" value="0.1" />
+    <xacro:property name="base_length" value="0.12" />
+    <xacro:property name="base_width" value="0.12" />
+    <xacro:property name="base_height" value="0.065" />
+    <xacro:property name="base_offset" value="0.02" />
+    <!-- arbitrary value for wheel value -->
+    <xacro:property name="wheel_mass" value="0.06" />
+    <xacro:property name="wheel_len" value="0.024" />
+    <xacro:property name="wheel_radius" value="0.035" />
+    <!-- Space btw top of beam and the each joint -->
+    <xacro:property name="z_offset" value="${base_height/2}" />
+    <!-- arbitrary value for ultrasonic eye value -->
+    <xacro:property name="sonic_mass" value="0.06" />
+    <xacro:property name="sonic_len" value="0.007" />
+    <xacro:property name="sonic_radius" value="0.0075" />
+    <!-- arbitrary value for front camera value -->
+    <xacro:property name="cam_length" value="0.02" />
+    <xacro:property name="cam_width" value="0.045" />
+    <xacro:property name="cam_height" value="0.033" />
+    <!-- Base Link -->
+    <link
+      name="base_link">
+    </link>
+    <!-- Base Footprint Joint -->
+    <joint name="base_footprint_joint" type="fixed">
+        <parent link="base_link"/>
+        <child link="base_footprint"/>
+        <origin xyz="0 0 0" rpy="0 0 0"/>
+    </joint>
+    <link
+      name="base_footprint">
+    </link>
+    <!-- Chassis Joint -->
+    <joint name="chassis_joint" type="fixed">
+        <parent link="base_link"/>
+        <child link="chassis"/>
+        <origin xyz="0 0 ${base_offset + z_offset}"/>
+    </joint>
+    <!-- Chassis Link-->
+    <link name="chassis">
+      <visual>
+        <origin xyz="0 0 0" rpy="0 0 0"/>
+        <geometry>
+          <box size="${base_length} ${base_width} ${base_height}"/>
+        </geometry>
+        <material name="black"/>
+      </visual>
+      <collision>
+        <origin xyz="0 0 0" rpy="0 0 0"/>
+        <geometry>
+          <box size="${base_length} ${base_width} ${base_height}"/>
+        </geometry>
+      </collision>
+      <inertial>
+        <origin xyz="0 0 0" rpy="0 0 0"/>
+        <mass value="${base_mass}"/>
+        <inertia
+          ixx="${base_mass / 12.0 * (base_length*base_length + base_height*base_height)}" ixy="0.0" ixz="0.0"
+          iyy="${base_mass / 12.0 * (base_height*base_height + base_width*base_width)}" iyz="0.0"
+          izz="${base_mass / 12.0 * (base_width*base_width + base_length*base_length)}"/>
       </inertial>
-  </link>
-  <!-- left wheel dummy Joint -->
-  <joint name="${prefix}left_wheel_dummy_joint" type="fixed">
-    <parent link="${prefix}chassis"/>
-    <child link="${prefix}left_wheel_dummy"/>
-    <origin xyz="-0.055 ${base_width/2 + wheel_len/2} ${base_offset-wheel_radius}" rpy="0 0 0"/>
-    <axis xyz="0 1 0"/>
-    <dynamics damping="0.2"/>
-  </joint>
-  <!-- left wheel dummy Link -->
-  <link name="${prefix}left_wheel_dummy">
-    <collision>
-      <origin xyz="0 0 0" rpy="0 0 0"/>
-      <geometry>
-        <cylinder length="${wheel_len}" radius="${wheel_radius}"/>
-      </geometry>
-    </collision>
-    <visual>
-      <origin xyz="0 0 0" rpy="${pi/2} 0 0"/>
-      <geometry>
-        <cylinder length="${wheel_len}" radius="${wheel_radius}"/>
-      </geometry>
-      <material name="orange"/>
-    </visual>
-    <inertial>
-      <origin xyz="0 0 0" rpy="0 0 0"/>
-      <mass value="${wheel_mass}"/>
-      <inertia
-        ixx="${wheel_mass / 12.0 * (3*wheel_radius + wheel_len*wheel_len)}" ixy="0.0" ixz="0.0"
-        iyy="${wheel_mass / 12.0 * wheel_radius*wheel_radius}" iyz="0.0"
-        izz="${wheel_mass / 12.0 * wheel_radius*wheel_radius}"/>
-      </inertial>
-  </link>
-  <!-- right wheel Joint -->
-    <joint name="${prefix}right_wheel_joint" type="continuous">
-    <parent link="${prefix}chassis"/>
-    <child link="${prefix}right_wheel"/>
-    <origin xyz="0.035 -${base_width/2 + wheel_len/2} ${base_offset-wheel_radius}" rpy="0 0 0"/>
-    <axis xyz="0 1 0"/>
-    <dynamics damping="0.2"/>
-  </joint>
-  <!-- right wheel Link -->
-  <link name="${prefix}right_wheel">
-    <collision>
-      <origin xyz="0 0 0" rpy="0 0 0"/>
-      <geometry>
-        <cylinder length="${wheel_len}" radius="${wheel_radius}"/>
-      </geometry>
-    </collision>
-    <visual>
-      <origin xyz="0 0 0" rpy="${pi/2} 0 0"/>
-      <geometry>
-        <cylinder length="${wheel_len}" radius="${wheel_radius}"/>
-      </geometry>
-      <material name="orange"/>
-    </visual>
-    <inertial>
-      <origin xyz="0 0 0" rpy="0 0 0"/>
-      <mass value="${wheel_mass}"/>
-      <inertia
-        ixx="${wheel_mass / 12.0 * (3*wheel_radius + wheel_len*wheel_len)}" ixy="0.0" ixz="0.0"
-        iyy="${wheel_mass / 12.0 * wheel_radius*wheel_radius}" iyz="0.0"
-        izz="${wheel_mass / 12.0 * wheel_radius*wheel_radius}"/>
-      </inertial>
-  </link>
-<!-- right wheel dummy Joint -->
-    <joint name="${prefix}right_wheel_dummy_joint" type="fixed">
-    <parent link="${prefix}chassis"/>
-    <child link="${prefix}right_wheel_dummy"/>
-    <origin xyz="-0.055 -${base_width/2 + wheel_len/2} ${base_offset-wheel_radius}" rpy="0 0 0"/>
-    <axis xyz="0 1 0"/>
-    <dynamics damping="0.2"/>
-  </joint>
-  <!-- right wheel dummy Link -->
-  <link name="${prefix}right_wheel_dummy">
-    <collision>
-      <origin xyz="0 0 0" rpy="0 0 0"/>
-      <geometry>
-        <cylinder length="${wheel_len}" radius="${wheel_radius}"/>
-      </geometry>
-    </collision>
-    <visual>
-      <origin xyz="0 0 0" rpy="${pi/2} 0 0"/>
-      <geometry>
-        <cylinder length="${wheel_len}" radius="${wheel_radius}"/>
-      </geometry>
-      <material name="orange"/>
-    </visual>
-    <inertial>
-      <origin xyz="0 0 0" rpy="0 0 0"/>
-      <mass value="${wheel_mass}"/>
-      <inertia
-        ixx="${wheel_mass / 12.0 * (3*wheel_radius + wheel_len*wheel_len)}" ixy="0.0" ixz="0.0"
-        iyy="${wheel_mass / 12.0 * wheel_radius*wheel_radius}" iyz="0.0"
-        izz="${wheel_mass / 12.0 * wheel_radius*wheel_radius}"/>
-      </inertial>
-  </link>
-  <!-- left ultrasonic eye Joint -->
-    <joint name="${prefix}left_ultrasonic_eye_joint" type="fixed">
-    <parent link="${prefix}chassis"/>
-    <child link="${prefix}left_ultrasonic_eye"/>
-    <origin xyz="0.06 0.0125 -0.0125" rpy="0 0 0"/>
-    <axis xyz="0 1 0"/>
-    <dynamics damping="0.2"/>
-  </joint>
-  <!-- left ultrasonic eye Link -->
-  <link name="${prefix}left_ultrasonic_eye">
-    <collision>
-      <origin xyz="0 0 0" rpy="0 0 0"/>
-      <geometry>
-        <cylinder length="0.007" radius="0.0075"/>
-      </geometry>
-    </collision>
-    <visual>
-      <origin xyz="0 0 0" rpy="0 ${pi/2} 0"/>
-      <geometry>
-        <cylinder length="${sonic_len}" radius="${sonic_radius}"/>
-      </geometry>
-      <material name="grey"/>
-    </visual>
-  </link>
-  <!-- right ultrasonic eye Joint -->
-  <joint name="${prefix}right_ultrasonic_eye_joint" type="fixed">
-    <parent link="${prefix}chassis"/>
-    <child link="${prefix}right_ultrasonic_eye"/>
-    <origin xyz="0.06 -0.0125 -0.0125" rpy="0 0 0"/>
-    <axis xyz="0 1 0"/>
-    <dynamics damping="0.2"/>
-  </joint>
-  <!-- right ultrasonic eye Link -->
-  <link name="${prefix}right_ultrasonic_eye">
-    <collision>
-      <origin xyz="0 0 0" rpy="0 0 0"/>
-      <geometry>
-        <cylinder length="${sonic_len}" radius="${sonic_radius}"/>
-      </geometry>
-    </collision>
-    <visual>
-      <origin xyz="0 0 0" rpy="0 ${pi/2} 0"/>
-      <geometry>
-        <cylinder length="0.007" radius="0.0075"/>
-      </geometry>
-      <material name="grey"/>
-    </visual>
-  </link>
+    </link>
+    <!-- left wheel Joint -->
+      <joint name="left_wheel_joint" type="continuous">
+      <parent link="chassis"/>
+      <child link="left_wheel"/>
+      <origin xyz="0.035 ${base_width/2 + wheel_len/2} ${base_offset-wheel_radius}" rpy="0 0 0"/>
+      <axis xyz="0 1 0"/>
+      <dynamics damping="0.2"/>
+    </joint>
+    <!-- left wheel Link -->
+    <link name="left_wheel">
+      <collision>
+        <origin xyz="0 0 0" rpy="0 0 0"/>
+        <geometry>
+          <cylinder length="${wheel_len}" radius="${wheel_radius}"/>
+        </geometry>
+      </collision>
+      <visual>
+        <origin xyz="0 0 0" rpy="${pi/2} 0 0"/>
+        <geometry>
+          <cylinder length="${wheel_len}" radius="${wheel_radius}"/>
+        </geometry>
+        <material name="orange"/>
+      </visual>
+      <inertial>
+        <origin xyz="0 0 0" rpy="0 0 0"/>
+        <mass value="${wheel_mass}"/>
+        <inertia
+          ixx="${wheel_mass / 12.0 * (3*wheel_radius + wheel_len*wheel_len)}" ixy="0.0" ixz="0.0"
+          iyy="${wheel_mass / 12.0 * wheel_radius*wheel_radius}" iyz="0.0"
+          izz="${wheel_mass / 12.0 * wheel_radius*wheel_radius}"/>
+        </inertial>
+    </link>
+    <!-- left wheel dummy Joint -->
+    <joint name="left_wheel_dummy_joint" type="fixed">
+      <parent link="chassis"/>
+      <child link="left_wheel_dummy"/>
+      <origin xyz="-0.055 ${base_width/2 + wheel_len/2} ${base_offset-wheel_radius}" rpy="0 0 0"/>
+      <axis xyz="0 1 0"/>
+      <dynamics damping="0.2"/>
+    </joint>
+    <!-- left wheel dummy Link -->
+    <link name="left_wheel_dummy">
+      <collision>
+        <origin xyz="0 0 0" rpy="0 0 0"/>
+        <geometry>
+          <cylinder length="${wheel_len}" radius="${wheel_radius}"/>
+        </geometry>
+      </collision>
+      <visual>
+        <origin xyz="0 0 0" rpy="${pi/2} 0 0"/>
+        <geometry>
+          <cylinder length="${wheel_len}" radius="${wheel_radius}"/>
+        </geometry>
+        <material name="orange"/>
+      </visual>
+      <inertial>
+        <origin xyz="0 0 0" rpy="0 0 0"/>
+        <mass value="${wheel_mass}"/>
+        <inertia
+          ixx="${wheel_mass / 12.0 * (3*wheel_radius + wheel_len*wheel_len)}" ixy="0.0" ixz="0.0"
+          iyy="${wheel_mass / 12.0 * wheel_radius*wheel_radius}" iyz="0.0"
+          izz="${wheel_mass / 12.0 * wheel_radius*wheel_radius}"/>
+        </inertial>
+    </link>
+    <!-- right wheel Joint -->
+      <joint name="right_wheel_joint" type="continuous">
+      <parent link="chassis"/>
+      <child link="right_wheel"/>
+      <origin xyz="0.035 -${base_width/2 + wheel_len/2} ${base_offset-wheel_radius}" rpy="0 0 0"/>
+      <axis xyz="0 1 0"/>
+      <dynamics damping="0.2"/>
+    </joint>
+    <!-- right wheel Link -->
+    <link name="right_wheel">
+      <collision>
+        <origin xyz="0 0 0" rpy="0 0 0"/>
+        <geometry>
+          <cylinder length="${wheel_len}" radius="${wheel_radius}"/>
+        </geometry>
+      </collision>
+      <visual>
+        <origin xyz="0 0 0" rpy="${pi/2} 0 0"/>
+        <geometry>
+          <cylinder length="${wheel_len}" radius="${wheel_radius}"/>
+        </geometry>
+        <material name="orange"/>
+      </visual>
+      <inertial>
+        <origin xyz="0 0 0" rpy="0 0 0"/>
+        <mass value="${wheel_mass}"/>
+        <inertia
+          ixx="${wheel_mass / 12.0 * (3*wheel_radius + wheel_len*wheel_len)}" ixy="0.0" ixz="0.0"
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