Commit message: 051023

File: src/kssbot/kssbot_description/ros2_control/kssbot.ros2_control.xacro (robot description, xacro)
@@ -13,6 +13,6 @@
           <joint name="left_wheel_joint">
             <command_interface name="velocity">
-              <param name="min">-10</param>
-              <param name="max">10</param>
+              <param name="min">-1</param>
+              <param name="max">1</param>
             </command_interface>
             <state_interface name="position"/>
@@ -21,6 +21,6 @@
           <joint name="right_wheel_joint">
             <command_interface name="velocity">
-              <param name="min">-10</param>
-              <param name="max">10</param>
+              <param name="min">-1</param>
+              <param name="max">1</param>
             </command_interface>
             <state_interface name="position"/>
@@ -36,6 +36,6 @@
             <joint name="left_wheel_joint">
                 <command_interface name="velocity">
-                    <param name="min">-10</param>
-                    <param name="max">10</param>
+                    <param name="min">-1</param>
+                    <param name="max">1</param>
                 </command_interface>
                 <state_interface name="velocity"/>
@@ -44,6 +44,6 @@
             <joint name="right_wheel_joint">
                 <command_interface name="velocity">
-                    <param name="min">-10</param>
-                    <param name="max">10</param>
+                    <param name="min">-1</param>
+                    <param name="max">1</param>
                 </command_interface>
                 <state_interface name="velocity"/>

File: src/kssbot/kssbot_description/urdf/kssbot_description.urdf copy.xacro (robot description, xacro)
@@ -5,11 +5,11 @@
     <xacro:property name="PI" value="3.1415926535897931"/>
     <!-- arbitrary value for base value -->
-    <xacro:property name="base_mass" value="5.0" />
+    <xacro:property name="base_mass" value="1.0" />
     <xacro:property name="base_length" value="0.12" />
     <xacro:property name="base_width" value="0.12" />
     <xacro:property name="base_height" value="0.065" />
-    <xacro:property name="base_z_offset" value="0.02" />
+    <xacro:property name="base_offset" value="0.02" />
     <!-- arbitrary value for wheel value -->
-    <xacro:property name="wheel_mass" value="0.5" />
+    <xacro:property name="wheel_mass" value="0.05" />
     <xacro:property name="wheel_len" value="0.024" />
     <xacro:property name="wheel_radius" value="0.035" />
@@ -41,5 +41,5 @@
         <parent link="base_link"/>
         <child link="chassis"/>
-        <origin xyz="0 0 ${base_z_offset + z_offset}"/>
+        <origin xyz="0 0 ${base_offset + z_offset}"/>
     </joint>
     <!-- Chassis Link-->
@@ -71,5 +71,5 @@
       <parent link="chassis"/>
       <child link="left_wheel"/>
-      <origin xyz="0.035 ${base_width/2 + wheel_len/2} ${base_z_offset-wheel_radius}" rpy="-${PI/2} 0 0"/>
+      <origin xyz="0.035 ${base_width/2 + wheel_len/2} ${base_offset-wheel_radius}" rpy="-${PI/2} 0 0"/>
       <axis xyz="0 0 1"/>
       <dynamics damping="0.2"/>
@@ -94,7 +94,7 @@
         <mass value="${wheel_mass}"/>
         <inertia
-          ixx="${wheel_mass / 12.0 * (3*wheel_radius* wheel_radius + wheel_len*wheel_len)}" ixy="0.0" ixz="0.0"
-          iyy="${wheel_mass / 12.0 * (3*wheel_radius* wheel_radius + wheel_len*wheel_len)}" iyz="0.0"
-          izz="${wheel_mass / 2.0 * wheel_radius*wheel_radius}"/>
+          ixx="${wheel_mass / 12.0 * (3*wheel_radius + wheel_len*wheel_len)}" ixy="0.0" ixz="0.0"
+          iyy="${wheel_mass / 12.0 * wheel_radius*wheel_radius}" iyz="0.0"
+          izz="${wheel_mass / 12.0 * wheel_radius*wheel_radius}"/>
       </inertial>
     </link>
@@ -103,5 +103,5 @@
       <parent link="chassis"/>
       <child link="left_wheel_dummy"/>
-      <origin xyz="-0.055 ${base_width/2 + wheel_len/2} ${base_z_offset-wheel_radius}" rpy="-${PI/2} 0 0"/>
+      <origin xyz="-0.055 ${base_width/2 + wheel_len/2} ${base_offset-wheel_radius}" rpy="-${PI/2} 0 0"/>
       <axis xyz="0 0 1"/>
       <dynamics damping="0.2"/>
@@ -126,8 +126,8 @@
         <mass value="${wheel_mass}"/>
         <inertia
-          ixx="${wheel_mass / 12.0 * (3*wheel_radius* wheel_radius + wheel_len*wheel_len)}" ixy="0.0" ixz="0.0"
-          iyy="${wheel_mass / 12.0 * (3*wheel_radius* wheel_radius + wheel_len*wheel_len)}" iyz="0.0"
-          izz="${wheel_mass / 2.0 * wheel_radius*wheel_radius}"/>
-        </inertial>
+          ixx="${wheel_mass / 12.0 * (3*wheel_radius + wheel_len*wheel_len)}" ixy="0.0" ixz="0.0"
+          iyy="${wheel_mass / 12.0 * wheel_radius*wheel_radius}" iyz="0.0"
+          izz="${wheel_mass / 12.0 * wheel_radius*wheel_radius}"/>
+      </inertial>
     </link>
     <!-- right wheel Joint -->
@@ -135,5 +135,5 @@
       <parent link="chassis"/>
       <child link="right_wheel"/>
-      <origin xyz="0.035 -${base_width/2 + wheel_len/2} ${base_z_offset-wheel_radius}" rpy="${PI/2} 0 0"/>
+      <origin xyz="0.035 -${base_width/2 + wheel_len/2} ${base_offset-wheel_radius}" rpy="${PI/2} 0 0"/>
       <axis xyz="0 0 -1"/>
       <dynamics damping="0.2"/>
@@ -158,7 +158,7 @@
         <mass value="${wheel_mass}"/>
         <inertia
-          ixx="${wheel_mass / 12.0 * (3*wheel_radius* wheel_radius + wheel_len*wheel_len)}" ixy="0.0" ixz="0.0"
-          iyy="${wheel_mass / 12.0 * (3*wheel_radius* wheel_radius + wheel_len*wheel_len)}" iyz="0.0"
-          izz="${wheel_mass / 2.0 * wheel_radius*wheel_radius}"/>
+          ixx="${wheel_mass / 12.0 * (3*wheel_radius + wheel_len*wheel_len)}" ixy="0.0" ixz="0.0"
+          iyy="${wheel_mass / 12.0 * wheel_radius*wheel_radius}" iyz="0.0"
+          izz="${wheel_mass / 12.0 * wheel_radius*wheel_radius}"/>
         </inertial>
     </link>
@@ -167,5 +167,5 @@
       <parent link="chassis"/>
       <child link="right_wheel_dummy"/>
-      <origin xyz="-0.055 -${base_width/2 + wheel_len/2} ${base_z_offset-wheel_radius}" rpy="${PI/2} 0 0"/>
+      <origin xyz="-0.055 -${base_width/2 + wheel_len/2} ${base_offset-wheel_radius}" rpy="${PI/2} 0 0"/>
       <axis xyz="0 0 -1"/>
       <dynamics damping="0.2"/>
@@ -190,7 +190,7 @@
         <mass value="${wheel_mass}"/>
         <inertia
-          ixx="${wheel_mass / 12.0 * (3*wheel_radius* wheel_radius + wheel_len*wheel_len)}" ixy="0.0" ixz="0.0"
-          iyy="${wheel_mass / 12.0 * (3*wheel_radius* wheel_radius + wheel_len*wheel_len)}" iyz="0.0"
-          izz="${wheel_mass / 2.0 * wheel_radius*wheel_radius}"/>
+          ixx="${wheel_mass / 12.0 * (3*wheel_radius + wheel_len*wheel_len)}" ixy="0.0" ixz="0.0"
+          iyy="${wheel_mass / 12.0 * wheel_radius*wheel_radius}" iyz="0.0"
+          izz="${wheel_mass / 12.0 * wheel_radius*wheel_radius}"/>
         </inertial>
     </link>
