Commit message: 030523

File: src/kssbot/kssbot_description/urdf/kssbot_description.urdf.xacro (robot description, xacro)
@@ -4,14 +4,14 @@
   <!-- Constants for robot dimensions -->
   <xacro:property name="PI" value="3.1415926535897931"/>
-  <xacro:property name="base_mass" value="0.3" /> <!-- arbitrary value for base mass -->
-  <xacro:property name="base_width" value="0.1" />
-  <xacro:property name="base_length" value="0.1" />
-  <xacro:property name="base_height" value="0.05" />
-  <xacro:property name="wheel_mass" value="0.3" /> <!-- arbitrary value for wheel mass -->
-  <xacro:property name="wheel_len" value="0.020" />
-  <xacro:property name="wheel_radius" value="0.015" />
+  <xacro:property name="base_mass" value="0.1" /> <!-- arbitrary value for base mass -->
+  <xacro:property name="base_width" value="0.12" />
+  <xacro:property name="base_length" value="0.12" />
+  <xacro:property name="base_height" value="0.07" />
+  <xacro:property name="wheel_mass" value="0.05" /> <!-- arbitrary value for wheel mass -->
+  <xacro:property name="wheel_len" value="0.025" />
+  <xacro:property name="wheel_radius" value="0.035" />
   <xacro:property name="caster_wheel_mass" value="0.1" /> <!-- arbitrary value for caster wheel mass -->
   <xacro:property name="caster_wheel_radius" value="0.015" />
-  <xacro:property name="z_offset" value="-${base_height/2}" /> <!-- Space btw top of beam and the each joint -->
+  <xacro:property name="z_offset" value="0.02" /> <!-- Space btw top of beam and the each joint -->
   <!-- Base Link -->
   <link name="${prefix}base_link">
@@ -23,5 +23,5 @@
     </collision>
     <visual>
-      <origin xyz="0 0 ${base_height/2}" rpy="0 0 0"/>
+      <origin xyz="0 0 ${z_offset}" rpy="0 0 0"/>
       <geometry>
         <box size="${base_width} ${base_length} ${base_height}"/>
@@ -32,5 +32,5 @@
       <origin xyz="0 0 0" rpy="0 0 0"/>
       <mass value="${base_mass}"/>
-      <inertia
+      <inertiaz_offset
         ixx="${base_mass / 12.0 * (base_length*base_length + base_height*base_height)}" ixy="0.0" ixz="0.0"
         iyy="${base_mass / 12.0 * (base_height*base_height + base_width*base_width)}" iyz="0.0"
@@ -41,5 +41,5 @@
       <parent link="${prefix}base_link"/>
       <child link="${prefix}left_wheel"/>
-      <origin xyz="0 -${base_width/2} ${z_offset}" rpy="0 0 0"/>
+      <origin xyz="0.025 -${base_width/2} ${z_offset}" rpy="0 0 0"/>
       <axis xyz="0 1 0"/>
       <dynamics damping="0.2"/>

Commit message: 043023

File: src/kssbot/kssbot_description/urdf/kssbot_description.urdf.xacro (robot description, xacro)
@@ -5,5 +5,5 @@
   <xacro:property name="PI" value="3.1415926535897931"/>
   <!-- arbitrary value for base value -->
-  <xacro:property name="base_mass" value="0.06" />
+  <xacro:property name="base_mass" value="0.1" />
   <xacro:property name="base_length" value="0.12" />
   <xacro:property name="base_width" value="0.12" />
@@ -14,7 +14,4 @@
   <xacro:property name="wheel_len" value="0.024" />
   <xacro:property name="wheel_radius" value="0.035" />
-  <!-- arbitrary value for caster wheel value -->
-  <xacro:property name="caster_wheel_mass" value="0.1" />
-  <xacro:property name="caster_wheel_radius" value="0.015" />
   <!-- Space btw top of beam and the each joint -->
   <xacro:property name="z_offset" value="${base_height/2}" />

Commit message: 101423

File: src/kssbot/kssbot_description/urdf/kssbot_description.urdf.xacro (robot description, xacro)
@@ -4,10 +4,10 @@
     <!-- Constants for robot dimensions -->
     <xacro:property name="PI" value="3.1415926535897931"/>
-    <!-- arbitrary value for base value -->
-    <xacro:property name="base_mass" value="5.0" />
-    <xacro:property name="base_length" value="0.12" />
-    <xacro:property name="base_width" value="0.12" />
-    <xacro:property name="base_height" value="0.065" />
-    <xacro:property name="base_z_offset" value="0.02" />
+    <!-- arbitrary value for chassis value -->
+    <xacro:property name="chassis_mass" value="5.0" />
+    <xacro:property name="chassis_length" value="0.12" />
+    <xacro:property name="chassis_width" value="0.12" />
+    <xacro:property name="chassis_height" value="0.065" />
+    <xacro:property name="chassis_z_offset" value="0.02" />
     <!-- arbitrary value for wheel value -->
     <xacro:property name="wheel_mass" value="0.5" />
@@ -15,5 +15,5 @@
     <xacro:property name="wheel_radius" value="0.035" />
     <!-- Space btw top of beam and the each joint -->
-    <xacro:property name="z_offset" value="${base_height/2}" />
+    <xacro:property name="z_offset" value="${chassis_height/2}" />
     <!-- arbitrary value for ultrasonic eye value -->
     <xacro:property name="sonic_mass" value="0.06" />
@@ -41,5 +41,5 @@
         <parent link="base_link"/>
         <child link="chassis"/>
-        <origin xyz="0 0 ${base_z_offset + z_offset}"/>
+        <origin xyz="0 0 ${chassis_z_offset + z_offset}"/>
     </joint>
     <!-- Chassis Link-->
@@ -48,5 +48,5 @@
         <origin xyz="0 0 0" rpy="0 0 0"/>
         <geometry>
-          <box size="${base_length} ${base_width} ${base_height}"/>
+          <box size="${chassis_length} ${chassis_width} ${chassis_height}"/>
         </geometry>
         <material name="black"/>
@@ -55,14 +55,14 @@
         <origin xyz="0 0 0" rpy="0 0 0"/>
         <geometry>
-          <box size="${base_length} ${base_width} ${base_height}"/>
-        </geometry>
-      </collision>
-      <inertial>
-        <origin xyz="0 0 0" rpy="0 0 0"/>
-        <mass value="${base_mass}"/>
-        <inertia
-          ixx="${base_mass / 12.0 * (base_length*base_length + base_height*base_height)}" ixy="0.0" ixz="0.0"
-          iyy="${base_mass / 12.0 * (base_height*base_height + base_width*base_width)}" iyz="0.0"
-          izz="${base_mass / 12.0 * (base_width*base_width + base_length*base_length)}"/>
+          <box size="${chassis_length} ${chassis_width} ${chassis_height}"/>
+        </geometry>
+      </collision>
+      <inertial>
+        <origin xyz="0 0 0" rpy="0 0 0"/>
+        <mass value="${chassis_mass}"/>
+        <inertia
+          ixx="${chassis_mass / 12.0 * (chassis_length*chassis_length + chassis_height*chassis_height)}" ixy="0.0" ixz="0.0"
+          iyy="${chassis_mass / 12.0 * (chassis_height*chassis_height + chassis_width*chassis_width)}" iyz="0.0"
+          izz="${chassis_mass / 12.0 * (chassis_width*chassis_width + chassis_length*chassis_length)}"/>
       </inertial>
     </link>
@@ -71,5 +71,5 @@
       <parent link="chassis"/>
       <child link="left_wheel"/>
-      <origin xyz="0.035 ${base_width/2 + wheel_len/2} ${base_z_offset-wheel_radius}" rpy="-${PI/2} 0 0"/>
+      <origin xyz="0.035 ${chassis_width/2 + wheel_len/2} ${chassis_z_offset-wheel_radius}" rpy="-${PI/2} 0 0"/>
       <axis xyz="0 0 1"/>
       <dynamics damping="0.2"/>
@@ -103,5 +103,5 @@
       <parent link="chassis"/>
       <child link="left_wheel_dummy"/>
-      <origin xyz="-0.055 ${base_width/2 + wheel_len/2} ${base_z_offset-wheel_radius}" rpy="-${PI/2} 0 0"/>
+      <origin xyz="-0.055 ${chassis_width/2 + wheel_len/2} ${chassis_z_offset-wheel_radius}" rpy="-${PI/2} 0 0"/>
       <axis xyz="0 0 1"/>
       <dynamics damping="0.2"/>
@@ -135,5 +135,5 @@
       <parent link="chassis"/>
       <child link="right_wheel"/>
-      <origin xyz="0.035 -${base_width/2 + wheel_len/2} ${base_z_offset-wheel_radius}" rpy="${PI/2} 0 0"/>
+      <origin xyz="0.035 -${chassis_width/2 + wheel_len/2} ${chassis_z_offset-wheel_radius}" rpy="${PI/2} 0 0"/>
       <axis xyz="0 0 -1"/>
       <dynamics damping="0.2"/>
@@ -167,5 +167,5 @@
       <parent link="chassis"/>
       <child link="right_wheel_dummy"/>
-      <origin xyz="-0.055 -${base_width/2 + wheel_len/2} ${base_z_offset-wheel_radius}" rpy="${PI/2} 0 0"/>
+      <origin xyz="-0.055 -${chassis_width/2 + wheel_len/2} ${chassis_z_offset-wheel_radius}" rpy="${PI/2} 0 0"/>
       <axis xyz="0 0 -1"/>
       <dynamics damping="0.2"/>
